Commit message: :sparkles: Phase 4f 傾斜検知・動的障害物テスト環境・安全機能統合
- incline_monitor.py: 傾斜検知純粋ロジック (quaternion_to_rpy, evaluate_incline, should_stop)
- incline_monitor_node.py: ROS 2 アダプター (/imu → /cmd_vel_incline 緊急停止)
- test_incline_monitor.py: 17テスト追加 (全189テスト通過)
- URDF: IMU センサー + gz-sim-imu-system プラグイン追加
- sim_launch.py: /imu ブリッジ追加
- nav2_launch.py: incline_monitor_node 統合
- twist_mux: cmd_vel_incline (priority:30) 追加 (Gemini レビュー修正)
- slope_test.world: 10°/25° 傾斜面テスト環境
- dynamic_obstacles.world: VelocityControl 付き移動障害物
- incline_params.yaml: 警告15°/緊急25°

Co-Authored-By: Claude Opus 4.6 <noreply@anthropic.com>

File: weeder_ws/src/grass_chopper/urdf/robot_description.urdf.xacro (robot description, xacro)
@@ -285,4 +285,31 @@
   </gazebo>
   <!-- ================================================================== -->
+  <!-- IMUセンサー: 慣性計測装置 (Phase 4f: 傾斜検知)                   -->
+  <!-- ================================================================== -->
+  <link name="imu_link">
+    <xacro:box_inertia m="0.01" x="0.01" y="0.01" z="0.01"/>
+    <visual>
+      <geometry>
+        <box size="0.01 0.01 0.01"/>
+      </geometry>
+      <material name="dark_grey"/>
+    </visual>
+  </link>
+  <joint name="imu_joint" type="fixed">
+    <parent link="base_link"/>
+    <child link="imu_link"/>
+    <origin xyz="0 0 0" rpy="0 0 0"/>
+  </joint>
+  <!-- Gazebo Harmonic用 IMUセンサー設定 -->
+  <gazebo reference="imu_link">
+    <sensor name="imu_sensor" type="imu">
+      <always_on>true</always_on>
+      <update_rate>50</update_rate>
+      <visualize>false</visualize>
+      <topic>imu</topic>
+      <gz_frame_id>imu_link</gz_frame_id>
+    </sensor>
+  </gazebo>
+  <!-- ================================================================== -->
   <!-- Gazebo Harmonicプラグイン                                         -->
   <!-- ================================================================== -->
@@ -312,4 +339,11 @@
     </plugin>
   </gazebo>
+  <!-- IMU システムプラグイン -->
+  <!-- IMU センサーデータを計算・発行するためのプラグイン -->
+  <gazebo>
+    <plugin filename="gz-sim-imu-system"
+            name="gz::sim::systems::Imu">
+    </plugin>
+  </gazebo>
   <!-- 関節状態パブリッシャー -->
   <!-- 車輪の回転角度をROS 2に送信（robot_state_publisherが使用） -->
